File: doc/examples/simple_pnb/simple_pnb.kicad_pcb (KiCad board)
At the start: 2 copper layers, 30 x 25 mm, 5 parts, among them J1 Conn_01x02, Q1 G_DATAMATRIX-code-4x4mm*

Commit message: Update the example so custom tab symbols are used
Parts:
- added T1: Tab, prusa_other:Tab_2mm, F.Cu at (165.0, 110.0)
- added T2: Tab, prusa_other:Tab_2mm, F.Cu at (155.0, 120.0)
- added T3: Tab, prusa_other:Tab_2mm, F.Cu at (135.0, 110.0)
- added T4: Tab, prusa_other:Tab_2mm, F.Cu at (155.0, 95.0)
Changed lines of the file:
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@@
   (net 3 "Net-(F1-Pad2)")
   (net 4 "Net-(J1-Pad2)")
+  (footprint "prusa_other:Tab_2mm" (layer "F.Cu")
+    (at 155 95 -90)
+    (descr "A symbol representing annotation for tab placement")
+    (property "PnB" "dnf")
+    (property "Sheetfile" "simple_pnb.kicad_sch")
+    (property "Sheetname" "")
+    (property "exclude_from_bom" "")
+    (attr exclude_from_pos_files exclude_from_bom)
+    (fp_text reference "T4" (at 1 0) (layer "F.SilkS") hide
+      (effects (font (size 1 1) (thickness 0.15)))
+    )
+    (fp_text value "Tab" (at -4.75 -1 90) (layer "Dwgs.User")
+      (effects (font (size 1 1) (thickness 0.2)))
+    )
+    (fp_text user "KIKIT: width: 2mm" (at -4.75 0.75 90) (layer "Dwgs.User") hide
+      (effects (font (size 0.5 0.5) (thickness 0.1)))
+    )
+    (fp_line (start 0 0) (end -1 1) (layer "Dwgs.User") (width 0.3))
+    (fp_line (start 0 1) (end 0 -1) (layer "Dwgs.User") (width 0.3))
+    (fp_line (start 0 0) (end -1 -1) (layer "Dwgs.User") (width 0.3))
+    (fp_line (start 0 0) (end -3 0) (layer "Dwgs.User") (width 0.3))
+  )
   (footprint "Resistor_SMD:R_0603_1608Metric" (layer "F.Cu")
     (at 155 100)
     (descr "Resistor SMD 0603 (1608 Metric), square (rectangular) end terminal, IPC_7351 nominal, (Body size source: IPC-SM-782 page 72, https://www.pcb-3d.com/wordpress/wp-content/uploads/ipc-sm-782a_amendment_1_and_2.pdf), generated with kicad-footprint-generator")
     (tags "resistor")
-    (property "Sheetfile" "simple_pnb.kicad_sch")
-    (property "Sheetname" "")
-    (property "id" "1")
+    (property "ID" "1")
+    (property "Sheetfile" "simple_pnb.kicad_sch")
+    (property "Sheetname" "")
     (attr smd)
     (fp_text reference "R1" (at 0 -1.43) (layer "F.SilkS")
@@
       (rotate (xyz 0 0 0))
     )
+  )
+  (footprint "prusa_other:Tab_2mm" (layer "F.Cu")
+    (at 135 110)
+    (descr "A symbol representing annotation for tab placement")
+    (property "PnB" "dnf")
+    (property "Sheetfile" "simple_pnb.kicad_sch")
+    (property "Sheetname" "")
+    (property "exclude_from_bom" "")
+    (attr exclude_from_pos_files exclude_from_bom)
+    (fp_text reference "T3" (at 1 0 90) (layer "F.SilkS") hide
+      (effects (font (size 1 1) (thickness 0.15)))
+    )
+    (fp_text value "Tab" (at -4.75 -1) (layer "Dwgs.User")
+      (effects (font (size 1 1) (thickness 0.2)))
+    )
+    (fp_text user "KIKIT: width: 2mm" (at -4.75 0.75 180) (layer "Dwgs.User") hide
+      (effects (font (size 0.5 0.5) (thickness 0.1)))
+    )
+    (fp_line (start 0 0) (end -1 -1) (layer "Dwgs.User") (width 0.3))
+    (fp_line (start 0 0) (end -3 0) (layer "Dwgs.User") (width 0.3))
+    (fp_line (start 0 0) (end -1 1) (layer "Dwgs.User") (width 0.3))
+    (fp_line (start 0 1) (end 0 -1) (layer "Dwgs.User") (width 0.3))
   )
   (footprint "Connector_PinHeader_2.54mm:PinHeader_1x02_P2.54mm_Horizontal" (layer "F.Cu")
@@
     (descr "car blade fuse direct solder")
     (tags "car blade fuse")
+    (property "ID" "3")
     (property "PnB" "#")
     (property "Sheetfile" "simple_pnb.kicad_sch")
     (property "Sheetname" "")
-    (property "id" "3")
     (attr through_hole)
     (fp_text reference "F1" (at 4.65 -3.9) (layer "F.SilkS")
@@
     )
   )
+  (footprint "prusa_other:Tab_2mm" (layer "F.Cu")
+    (at 155 120 90)
+    (descr "A symbol representing annotation for tab placement")
+    (property "PnB" "dnf")
+    (property "Sheetfile" "simple_pnb.kicad_sch")
+    (property "Sheetname" "")
+    (property "exclude_from_bom" "")
+    (attr exclude_from_pos_files exclude_from_bom)
+    (fp_text reference "T2" (at 1 0) (layer "F.SilkS") hide
+      (effects (font (size 1 1) (thickness 0.15)))
+    )
+    (fp_text value "Tab" (at -4.75 -1 90) (layer "Dwgs.User")
+      (effects (font (size 1 1) (thickness 0.2)))
+    )
+    (fp_text user "KIKIT: width: 2mm" (at -4.75 0.75 90) (layer "Dwgs.User") hide
+      (effects (font (size 0.5 0.5) (thickness 0.1)))
+    )
+    (fp_line (start 0 0) (end -1 1) (layer "Dwgs.User") (width 0.3))
+    (fp_line (start 0 0) (end -3 0) (layer "Dwgs.User") (width 0.3))
+    (fp_line (start 0 1) (end 0 -1) (layer "Dwgs.User") (width 0.3))
+    (fp_line (start 0 0) (end -1 -1) (layer "Dwgs.User") (width 0.3))
+  )
+  (footprint "prusa_other:Tab_2mm" (layer "F.Cu")
+    (at 165 110 180)
+    (descr "A symbol representing annotation for tab placement")
+    (property "PnB" "dnf")
+    (property "Sheetfile" "simple_pnb.kicad_sch")
+    (property "Sheetname" "")
+    (property "exclude_from_bom" "")
+    (attr exclude_from_pos_files exclude_from_bom)
+    (fp_text reference "T1" (at 1 0 90) (layer "F.SilkS") hide
+      (effects (font (size 1 1) (thickness 0.15)))
+    )
+    (fp_text value "Tab" (at -4.75 -1) (layer "Dwgs.User")
+      (effects (font (size 1 1) (thickness 0.2)))
+    )
+    (fp_text user "KIKIT: width: 2mm" (at -4.75 0.75) (layer "Dwgs.User") hide
+      (effects (font (size 0.5 0.5) (thickness 0.1)))
+    )
+    (fp_line (start 0 0) (end -1 -1) (layer "Dwgs.User") (width 0.3))
+    (fp_line (start 0 0) (end -3 0) (layer "Dwgs.User") (width 0.3))
+    (fp_line (start 0 0) (end -1 1) (layer "Dwgs.User") (width 0.3))
+    (fp_line (start 0 1) (end 0 -1) (layer "Dwgs.User") (width 0.3))
+  )
   (footprint "prusa_other:Datamatyrix-code-4x4mm" (layer "F.Cu")
     (at 140 112.5)
@@
     (descr "LED SMD 0603 (1608 Metric), square (rectangular) end terminal, IPC_7351 nominal, (Body size source: http://www.tortai-tech.com/upload/download/2011102023233369053.pdf), generated with kicad-footprint-generator")
     (tags "LED")
-    (property "Sheetfile" "simple_pnb.kicad_sch")
-    (property "Sheetname" "")
-    (property "id" "2")
+    (property "ID" "2")
+    (property "Sheetfile" "simple_pnb.kicad_sch")
+    (property "Sheetname" "")
     (attr smd)
     (fp_text reference "D1" (at 0 -1.43 90) (layer "F.SilkS")
